Commit message: wip: ball panda hardware demo

File: robust_value_approx/test/ball_panda_description/panda.urdf (robot description, URDF)
Before this commit: robot panda, 14 links, 13 joints
Joints:
- joint panda_paddle_target_joint: origin xyz=0 .005 .175 rpy=0 0 0 -> xyz=0.129, 0.002, 0.128 rpy=-3.064 -0.021 0.034; parent panda_paddle -> panda_hand
