Commit message: falling cubes dataset

File: neural_network_lyapunov/urdf/pendulum.urdf (robot description, URDF)
Before this commit: robot physics, 2 links, 1 joints
Joints:
- joint base_to_pole: limit (none) -> lower=-100 upper=100 effort=1000.0 velocity=100; type continuous -> prismatic

Commit message: fixes bug in pendulum urdf

File: neural_network_lyapunov/urdf/pendulum.urdf (robot description, URDF)
Before this commit: robot pendulum, 2 links, 1 joints
Joints:
- joint base_to_pole: limit lower=-100 upper=100 effort=1000.0 velocity=100 -> (none); type prismatic -> continuous

Commit message: training stable dynamics using lyapunov stability

File: neural_network_lyapunov/urdf/pendulum.urdf (robot description, URDF)
Before this commit: robot pendulum, 2 links, 1 joints
Links:
- link pole: mass 0.1 -> 1.
